File: NixiePhoton2Ctrl/NixiePhoton2Ctrl.kicad_pcb (KiCad board)
At the start: 2 copper layers, 90 x 70 mm, 11 parts, among them J1 DST Switch, J2 Main Board, J3 Rotary Encoder, U1 Particle_Photon2, U2 DS3231RTC

Commit message: misc
Parts:
- removed ? (x4): , MountingHole:MountingHole_3.2mm_M3

Commit message: misc
Parts:
- R1, R2: value 2K -> 4K7; footprint Resistor_THT:R_Axial_DIN0204_L3.6mm_D1.6mm_P5.08mm_Horizontal -> Resistor_THT:R_Axial_DIN0207_L6.3mm_D2.5mm_P7.62mm_Horizontal
- moved R1 2.08 mm to (126.0, 129.0)
Connections:
- R1 pad 1: +5V -> +3V3
- R2 pad 1: +5V -> +3V3
- U1 pad 1: Net-(U1-Pad1) -> unconnected-(U1-~{RST}-Pad1)
- U1 pad 10: RPB -> unconnected-(U1-S3-Pad10)
- U1 pad 13: Net-(U1-Pad13) -> unconnected-(U1-MISO-Pad13)
- U1 pad 14: Net-(U1-Pad14) -> unconnected-(U1-RX-Pad14)
- U1 pad 15: Net-(U1-Pad15) -> unconnected-(U1-TX-Pad15)
- U1 pad 16: Net-(U1-Pad16) -> unconnected-(U1-NC-Pad16)
- U1 pad 19: Net-(U1-Pad19) -> unconnected-(U1-D2-Pad19)
- U1 pad 2: Net-(U1-Pad2) -> +3V3
- U1 pad 20: Net-(U1-Pad20) -> unconnected-(U1-D3-Pad20)
- U1 pad 21: Net-(U1-Pad21) -> unconnected-(U1-D4-Pad21)
- U1 pad 22: Net-(U1-Pad22) -> RPB
- U1 pad 25: Net-(U1-Pad25) -> unconnected-(U1-D10-Pad25)
- U1 pad 27: Net-(U1-Pad27) -> unconnected-(U1-EN-Pad27)
- U1 pad 28: Net-(U1-Pad28) -> unconnected-(U1-LI+-Pad28)
- U1 pad 3: Net-(U1-Pad3) -> unconnected-(U1-~{Mode}-Pad3)
- U1 pad 5: Net-(U1-Pad5) -> unconnected-(U1-A0-Pad5)
- U1 pad 6: Net-(U1-Pad6) -> unconnected-(U1-A1-Pad6)
- U2 pad 1: +5V -> +3V3
- U2 pad 5: Net-(U2-Pad5) -> unconnected-(U2-Bat-Pad5)
- U2 pad 6: Net-(U2-Pad6) -> unconnected-(U2-32K-Pad6)
- U2 pad 7: Net-(U2-Pad7) -> unconnected-(U2-SQW-Pad7)
- U2 pad 8: Net-(U2-Pad8) -> unconnected-(U2-~{RST}-Pad8)
Routing:
- net +5V: track 0.00 -> 92.0 mm
- net RPB: track 33.0 -> 41.0 mm
- net SDA: track 43.4 -> 40.7 mm
- net SCL: track 41.4 -> 39.0 mm
- added copper zone on F.Cu, net +3V3
- removed copper zone on F.Cu, net +5V
Other:
- net class Default removed
- board text added: "Nixie Controller Rev B Dec 2023 D. McQ"
- board text removed: "Nixie Controller Rev A Dec 2023 D. McQ"
